Commit message: Have working kinova_jaco.urdf file now!

File: src/nrc/kinova_jaco.urdf (robot description, URDF)
Before this commit: robot kinova_jaco, 8 links, 7 joints
Links:
- removed link link6
- link base_link: geometry visual mesh filename=kinova_jaco_graphics/base.obj scale=0.001 0.001 0.001; visual mesh filename=kinova_jaco_graphics/ring-large.obj scale=0.001 0.001 0.001
- link link0: mass 4 -> 0.8; geometry visual mesh filename=kinova_jaco_graphics/link0.obj scale=0.001 0.001 0.001; visual mesh filename=kinova_jaco_graphics/ring-large.obj scale=0.001 0.001 0.001
- link link1: mass 4 -> 0.85; geometry visual mesh filename=kinova_jaco_graphics/link1.obj scale=0.001 0.001 0.001; visual mesh filename=kinova_jaco_graphics/ring-large.obj scale=0.001 0.001 0.001
- link link2: mass 4 -> 0.85; geometry visual mesh filename=kinova_jaco_graphics/link2.obj scale=0.001 0.001 0.001; visual mesh filename=kinova_jaco_graphics/ring-small.obj scale=0.001 0.001 0.001
- link link3: mass 4 -> 0.85; geometry visual mesh filename=kinova_jaco_graphics/link3.obj scale=0.001 0.001 0.001; visual mesh filename=kinova_jaco_graphics/ring-small-rot45.obj scale=0.001 0.001 0.001
- link link4: mass 3 -> 0.85; geometry visual mesh filename=kinova_jaco_graphics/link4.obj scale=0.001 0.001 0.001; visual mesh filename=kinova_jaco_graphics/ring-small-rot45.obj scale=0.001 0.001 0.001
- link link5: mass 2 -> 0.727; geometry collision mesh filename=kinova_jaco_graphics/link5-hand-base.obj scale=0.001 0.001 0.001; visual mesh filename=kinova_jaco_graphics/finger0-opposed.obj scale=0.001 0.001 0.001
Joints:
- removed joint j6
- joint j0: limit lower=-2.967 upper=2.967 effort=176 velocity=1.7104 -> lower=-20 upper=20 effort=97.6 velocity=2; origin xyz=0.000000 0.000000 0.155767 rpy=0.000000 0.000000 0.000000 -> xyz=0.000000 0.000000 0.1575 rpy=0.000000 0.000000 0.000000
- joint j1: axis 0 1 0 -> 1 0 0; limit lower=-2.0944 upper=2.0944 effort=176 velocity=1.7104 -> lower=-20 upper=20 effort=186.4 velocity=2; origin xyz=0.000000 0.000000 0.182500 rpy=0.000000 0.000000 0.000000 -> xyz=0.000000 0.000000 0.118 rpy=0.000000 0.000000 0.000000
- joint j2: axis 0 0 1 -> 1 0 0; limit lower=-2.967 upper=2.967 effort=110 velocity=1.7453 -> lower=-20 upper=20 effort=186.4 velocity=2; origin xyz=0.000000 0.000000 0.185000 rpy=0.000000 0.000000 0.000000 -> xyz=0.000000 0.000000 0.41 rpy=0.000000 0.000000 0.000000
- joint j3: axis 0 1 0 -> 0 0 1; limit lower=-2.0944 upper=2.0944 effort=110 velocity=2.2689 -> lower=-20 upper=20 effort=186.4 velocity=2; origin xyz=0.000000 0.000000 0.217000 rpy=0.000000 0.000000 3.1415926535897 -> xyz=0.0098 0.0 0.2073 rpy=0.000000 0.000000 0.000000
- joint j4: limit lower=-2.967 upper=2.967 effort=110 velocity=2.4434 -> lower=-20 upper=20 effort=186.4 velocity=2; origin xyz=0.000000 0.000000 0.186000 rpy=0.000000 0.000000 -3.1415926535897 -> xyz=0.0 -0.03705 0.064172 rpy=1.0471975512 0.000000 0.000000
- joint j5: axis 0 1 0 -> 0 0 1; limit lower=-2.0944 upper=2.0944 effort=40 velocity=3.1416 -> lower=-20 upper=20 effort=186.4 velocity=2; origin xyz=0.000000 0.000000 0.217003 rpy=0.000000 0.000000 0.000000 -> xyz=0.0 -0.03705 0.064172 rpy=1.0471975512 0.000000 0.000000

Commit message: Robot controller with Kinova works!

File: src/nrc/kinova_jaco.urdf (robot description, URDF)
Before this commit: robot kinova_jaco, 7 links, 6 joints
Joints:
- joint j0: limit lower=-20 upper=20 effort=97.6 velocity=2 -> lower=-20 upper=20 effort=97.6 velocity=4
- joint j1: limit lower=-20 upper=20 effort=186.4 velocity=2 -> lower=-20 upper=20 effort=186.4 velocity=4
- joint j2: limit lower=-20 upper=20 effort=186.4 velocity=2 -> lower=-20 upper=20 effort=186.4 velocity=4
- joint j3: limit lower=-20 upper=20 effort=186.4 velocity=2 -> lower=-20 upper=20 effort=186.4 velocity=4
- joint j4: limit lower=-20 upper=20 effort=186.4 velocity=2 -> lower=-20 upper=20 effort=186.4 velocity=4
- joint j5: limit lower=-20 upper=20 effort=186.4 velocity=2 -> lower=-20 upper=20 effort=186.4 velocity=4
